File: TKL_Video/TKL_Video.kicad_sch (KiCad schematic)
At the start: 229 parts, among them J1 USB_C_Receptacle_USB2.0, J2 Conn_01x04, J3 Conn_01x05, SW10 MX_SW_HS, SW100 MX_SW_HS, SW104 MX_SW_HS, SW105 MX_SW_HS, SW106 MX_SW_HS, SW107 MX_SW_HS, SW108 MX_SW_HS, SW109 MX_SW_HS, SW11 MX_SW_HS, SW110 MX_SW_HS, SW112 MX_SW_HS, SW113 MX_SW_HS, SW114 MX_SW_HS, SW115 MX_SW_HS, SW116 MX_SW_HS, SW117 MX_SW_HS, SW118 MX_SW_HS, SW12 MX_SW_HS, SW13 MX_SW_HS, SW14 MX_SW_HS, SW15 MX_SW_HS, SW16 MX_SW_HS, SW17 MX_SW_HS, SW18 MX_SW_HS, SW19 MX_SW_HS, SW20 MX_SW_HS, SW21 MX_SW_HS, SW22 MX_SW_HS, SW23 MX_SW_HS, SW24 MX_SW_HS, SW25 MX_SW_HS, SW26 MX_SW_HS, SW27 MX_SW_HS, SW28 MX_SW_HS, SW29 MX_SW_HS, SW3 MX_SW_HS, SW30 MX_SW_HS, SW31 MX_SW_HS, SW32 MX_SW_HS, SW33 MX_SW_HS, SW34 MX_SW_HS, SW35 MX_SW_HS, SW36 MX_SW_HS, SW37 MX_SW_HS, SW38 MX_SW_HS, SW39 MX_SW_HS, SW40 MX_SW_HS, SW41 MX_SW_HS, SW42 MX_SW_HS, SW43 MX_SW_HS, SW44 MX_SW_HS, SW45 MX_SW_HS, SW46 MX_SW_HS, SW47 MX_SW_HS, SW48 MX_SW_HS, SW49 MX_SW_HS, SW5 MX_SW_HS, SW50 MX_SW_HS, SW51 MX_SW_HS, SW52 MX_SW_HS, SW54 MX_SW_HS, SW55 MX_SW_HS, SW56 MX_SW_HS, SW57 MX_SW_HS, SW58 MX_SW_HS, SW59 MX_SW_HS, SW6 MX_SW_HS, SW60 MX_SW_HS, SW61 MX_SW_HS, SW62 MX_SW_HS, SW63 MX_SW_HS, SW64 MX_SW_HS, SW65 MX_SW_HS, SW66 MX_SW_HS, SW67 MX_SW_HS, SW68 MX_SW_HS, SW7 MX_SW_HS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

Commit message: Video Part 2
Parts:
- added C13, C14, C15, C16: 100n, Capacitor_SMD:C_0402_1005Metric, symbol Device:C_Small
Connections:
- net +1V1: now also C13.1
- net +3V3: now also J3.4 (Pin_4), C14.1, C15.1, C16.1; no longer J3.2 (Pin_2)
- net GND: now also J3.5 (Pin_5), C13.2, C14.2, C15.2, C16.2; no longer J3.3 (Pin_3)
- net RESET: now also J3.3 (Pin_3); no longer J3.1 (Pin_1)
- net SWC: now also J3.1 (Pin_1); no longer J3.4 (Pin_4)
- net SWD: now also J3.2 (Pin_2); no longer J3.5 (Pin_5)
- net at D110.2 (A), SW112.2: now also SW88.2
- net at D93.2 (A), SW95.2: now also SW74.1
- net at D98.2 (A), SW100.2: now also SW90.2
- net at SW100.1: now also SW90.1
- net at SW93.1: now also SW72.2
- net at D91.2 (A), SW93.2: now also SW72.1
- net at D113.2 (A): now also SW115.1; no longer SW115.2
- net at SW94.1: now also SW73.2
- net at D92.2 (A), SW94.2: now also SW73.1
- net at SW95.1: now also SW74.2
- net at SW116.1: now also SW75.1
- net at D114.2 (A), SW116.2: now also SW75.2
- net at D103.2 (A): now also SW105.1, SW92.2; no longer SW105.2
- net at SW34.1: now also SW13.1
- net at D32.2 (A), SW34.2: now also SW13.2
- net at SW107.1: now also D105.2 (A), SW118.2
- net at SW107.2: now also SW118.1; no longer D105.2 (A)
- net at SW92.1: now also SW105.2
- net at D55.2 (A): now also SW117.2, SW57.1; no longer SW57.2
- net at D33.2 (A): now also SW35.1; no longer SW35.2
- net at SW112.1: now also SW88.1
- net at SW117.1: now also SW57.2
- net at SW106.1: now also D104.2 (A), SW114.2
- net at SW106.2: now also SW114.1; no longer D104.2 (A)
Other:
- moved on the sheet: C10, C11, C12, C6, C7, C8, C9, D1, D10, D102, D103, D104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
